File: keyboard-1/keyboard-1.kicad_pcb (KiCad board)
At the start: 2 copper layers, 33 parts, among them SW1 SW_Push, SW10 SW_Push, SW11 SW_Push, SW12 SW_Push, SW13 SW_Push, SW14 SW_Push, SW15 SW_Push, SW16 SW_Push, SW17 SW_Push, SW18 SW_Push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

Commit message: put components on pcb
Parts:
- removed U1: Elite-C, Keebio-Parts:Elite-C
- added J1: Conn_01x12, Connector_PinHeader_2.54mm:PinHeader_1x12_P2.54mm_Vertical, F.Cu at (36.8, 58.4)
- added J2: Conn_01x12, Connector_PinHeader_2.54mm:PinHeader_1x12_P2.54mm_Vertical, F.Cu at (52.1, 58.4)
- added J3: Conn_01x04_Female, Connector_PinSocket_2.54mm:PinSocket_1x04_P2.54mm_Vertical, F.Cu at (40.6, 92.7)
- added U2: TRRS, Keebio-Parts:TRRS-PJ-320A, F.Cu at (61.0, 59.7)
Connections:
- net COL0 renamed /COL0
- net COL1 renamed /COL1
- net COL2 renamed /COL2
- net COL3 renamed /COL3
- net COL4 renamed /COL4
- net COL5 renamed /COL5
- net ROW0 renamed /ROW0
- net ROW1 renamed /ROW1
- net ROW2 renamed /ROW2
- net ROW3 renamed /ROW3

Commit message: traces to components
Routing:
- net /COL2: track 0.00 -> 276.0 mm
- net /COL1: track 0.00 -> 224.6 mm
- net /COL4: track 0.00 -> 188.7 mm
- net /COL5: track 0.00 -> 172.1 mm
- net /COL3: track 0.00 -> 160.6 mm
- net /ROW2: track 0.00 -> 138.3 mm
- net /ROW1: track 0.00 -> 122.8 mm
- net /ROW0: track 0.00 -> 110.6 mm
- net /COL0: track 0.00 -> 108.4 mm
- net /ROW3: track 0.00 -> 94.9 mm
- net GND: track 0.00 -> 37.2 mm
- net VCC: track 0.00 -> 31.5 mm
- net /SERIAL: track 0.00 -> 27.2 mm
- net /SDA: track 0.00 -> 26.7 mm
- net /SCL: track 0.00 -> 26.2 mm
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
Commit message: reset button + per key leds
Parts:
- removed J1, J2: Conn_01x12, Connector_PinHeader_2.54mm:PinHeader_1x12_P2.54mm_Vertical
- added D12: SK6812MINI, LED_SMD:LED_SK6812MINI_PLCC4_3.5x3.5mm_P1.75mm, F.Cu at (110.5, 142.2)
- added D13: SK6812MINI, LED_SMD:LED_SK6812MINI_PLCC4_3.5x3.5mm_P1.75mm, F.Cu at (121.1, 132.9)
- added D14: SK6812MINI, LED_SMD:LED_SK6812MINI_PLCC4_3.5x3.5mm_P1.75mm, F.Cu at (110.5, 147.3)
- added D15: SK6812MINI, LED_SMD:LED_SK6812MINI_PLCC4_3.5x3.5mm_P1.75mm, F.Cu at (117.5, 142.2)
- added D16: SK6812MINI, LED_SMD:LED_SK6812MINI_PLCC4_3.5x3.5mm_P1.75mm, F.Cu at (128.1, 132.9)
- added D17: SK6812MINI, LED_SMD:LED_SK6812MINI_PLCC4_3.5x3.5mm_P1.75mm, F.Cu at (110.5, 152.3)
- added D18: SK6812MINI, LED_SMD:LED_SK6812MINI_PLCC4_3.5x3.5mm_P1.75mm, F.Cu at (117.5, 147.3)
- added D19: SK6812MINI, LED_SMD:LED_SK6812MINI_PLCC4_3.5x3.5mm_P1.75mm, F.Cu at (124.5, 137.9)
- added D20: SK6812MINI, LED_SMD:LED_SK6812MINI_PLCC4_3.5x3.5mm_P1.75mm, F.Cu at (135.1, 132.9)
- added D21: SK6812MINI, LED_SMD:LED_SK6812MINI_PLCC4_3.5x3.5mm_P1.75mm, F.Cu at (124.5, 143.0)
- added D22: SK6812MINI, LED_SMD:LED_SK6812MINI_PLCC4_3.5x3.5mm_P1.75mm, F.Cu at (117.5, 152.3)
- added D23: SK6812MINI, LED_SMD:LED_SK6812MINI_PLCC4_3.5x3.5mm_P1.75mm, F.Cu at (131.6, 137.9)
- added D24: SK6812MINI, LED_SMD:LED_SK6812MINI_PLCC4_3.5x3.5mm_P1.75mm, F.Cu at (124.5, 148.0)
- added D25: SK6812MINI, LED_SMD:LED_SK6812MINI_PLCC4_3.5x3.5mm_P1.75mm, F.Cu at (142.2, 132.9)
- added D26: SK6812MINI, LED_SMD:LED_SK6812MINI_PLCC4_3.5x3.5mm_P1.75mm, F.Cu at (131.6, 143.0)
- added D27: SK6812MINI, LED_SMD:LED_SK6812MINI_PLCC4_3.5x3.5mm_P1.75mm, F.Cu at (138.6, 137.9)
- added D28: SK6812MINI, LED_SMD:LED_SK6812MINI_PLCC4_3.5x3.5mm_P1.75mm, F.Cu at (124.5, 153.1)
- added D29: SK6812MINI, LED_SMD:LED_SK6812MINI_PLCC4_3.5x3.5mm_P1.75mm, F.Cu at (131.6, 148.0)
- added D30: SK6812MINI, LED_SMD:LED_SK6812MINI_PLCC4_3.5x3.5mm_P1.75mm, F.Cu at (149.2, 132.9)
- added D31: SK6812MINI, LED_SMD:LED_SK6812MINI_PLCC4_3.5x3.5mm_P1.75mm, F.Cu at (138.6, 143.0)
- added D32: SK6812MINI, LED_SMD:LED_SK6812MINI_PLCC4_3.5x3.5mm_P1.75mm, F.Cu at (145.6, 137.9)
- added SW22: SW_Push, Keebio-Parts:SW_Tactile_SPST_Angled_MJTP1117, F.Cu at (36.8, 78.7)
- added U1: Elite-C, Keebio-Parts:Elite-C-castellated-24pin-holes, F.Cu at (53.3, 74.9)
- moved U2 22.9 mm to (38.1, 58.4)
- moved J3 8.89 mm to (49.5, 92.7)
Routing:
- net /COL1: track 224.6 -> 78.4 mm
- net /COL4: track 188.7 -> 50.1 mm
- net /COL5: track 172.1 -> 46.2 mm
- net /COL3: track 160.6 -> 47.4 mm
- net /COL2: track 276.0 -> 187.6 mm
- net /ROW3: track 94.9 -> 13.7 mm
- net /ROW2: track 138.3 -> 76.2 mm
- net /ROW1: track 122.8 -> 76.2 mm
- net GND: track 37.2 -> 0.00 mm
- net /ROW0: track 110.6 -> 76.2 mm
- net VCC: track 31.5 -> 0.00 mm
- net /SERIAL: track 27.2 -> 0.00 mm
- net /SDA: track 26.7 -> 0.00 mm
- net /SCL: track 26.2 -> 0.00 mm
- net /COL0: track 108.4 -> 84.9 mm
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