File: keyboard-1/keyboard-1.sch (KiCad schematic (older format))
At the start: 36 parts, among them SW1 SW_Push, SW10 SW_Push, SW11 SW_Push, SW12 SW_Push, SW13 SW_Push, SW14 SW_Push, SW15 SW_Push, SW16 SW_Push, SW17 SW_Push, SW18 SW_Push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

Commit message: put components on pcb
Parts:
- J1, J2: renamed from J?; footprint (none) -> Connector_PinHeader_2.54mm:PinHeader_1x12_P2.54mm_Vertical
- J3: renamed from J?; footprint Connector_PinSocket_2.54mm:PinSocket_1x01_P2.54mm_Vertical -> Connector_PinSocket_2.54mm:PinSocket_1x04_P2.54mm_Vertical
Changed lines of the file:
@@
 	5500 6000 5400 6000
 $Comp
-L Connector_Generic:Conn_01x12 J?
+L Connector_Generic:Conn_01x12 J1
 U 1 1 6044E7FE
 P 2450 5950
-F 0 "J?" H 2530 5942 50  0000 L CNN
+F 0 "J1" H 2530 5942 50  0000 L CNN
 F 1 "Conn_01x12" H 2530 5851 50  0000 L CNN
-F 2 "" H 2450 5950 50  0001 C CNN
+F 2 "Connector_PinHeader_2.54mm:PinHeader_1x12_P2.54mm_Vertical" H 2450 5950 50  0001 C CNN
 F 3 "~" H 2450 5950 50  0001 C CNN
 	1    2450 5950
@@
 $EndComp
 $Comp
-L Connector_Generic:Conn_01x12 J?
+L Connector_Generic:Conn_01x12 J2
 U 1 1 60456305
 P 3250 6050
-F 0 "J?" H 3168 5225 50  0000 C CNN
+F 0 "J2" H 3168 5225 50  0000 C CNN
 F 1 "Conn_01x12" H 3168 5316 50  0000 C CNN
-F 2 "" H 3250 6050 50  0001 C CNN
+F 2 "Connector_PinHeader_2.54mm:PinHeader_1x12_P2.54mm_Vertical" H 3250 6050 50  0001 C CNN
 F 3 "~" H 3250 6050 50  0001 C CNN
 	1    3250 6050
@@
 	3600 5950 3450 5950
 $Comp
-L Connector:Conn_01x04_Female J?
+L Connector:Conn_01x04_Female J3
 U 1 1 60477B7D
 P 5350 7400
-F 0 "J?" V 5196 7548 50  0000 L CNN
+F 0 "J3" V 5196 7548 50  0000 L CNN
 F 1 "Conn_01x04_Female" V 5287 7548 50  0000 L CNN
-F 2 "Connector_PinSocket_2.54mm:PinSocket_1x01_P2.54mm_Vertical" H 5350 7400 50  0001 C CNN
+F 2 "Connector_PinSocket_2.54mm:PinSocket_1x04_P2.54mm_Vertical" H 5350 7400 50  0001 C CNN
 F 3 "~" H 5350 7400 50  0001 C CNN
 	1    5350 7400
@@
 $EndComp
 $Comp
-L power:VCC #PWR?
+L power:VCC #PWR0101
 U 1 1 60479E6C
 P 5250 6900
-F 0 "#PWR?" H 5250 6750 50  0001 C CNN
+F 0 "#PWR0101" H 5250 6750 50  0001 C CNN
 F 1 "VCC" H 5265 7073 50  0000 C CNN
 F 2 "" H 5250 6900 50  0001 C CNN
@@
 $EndComp
 $Comp
-L power:GND #PWR?
+L power:GND #PWR0102
 U 1 1 6047AD0B
 P 4850 7200
-F 0 "#PWR?" H 4850 6950 50  0001 C CNN
+F 0 "#PWR0102" H 4850 6950 50  0001 C CNN
 F 1 "GND" H 4855 7027 50  0000 C CNN
 F 2 "" H 4850 7200 50  0001 C CNN
@@
 COL4
 $Comp
-L power:VCC #PWR?
+L power:VCC #PWR0105
 U 1 1 6048C43C
 P 4050 5650
-F 0 "#PWR?" H 4050 5500 50  0001 C CNN
+F 0 "#PWR0105" H 4050 5500 50  0001 C CNN
 F 1 "VCC" H 4065 5823 50  0000 C CNN
 F 2 "" H 4050 5650 50  0001 C CNN
@@
 $EndComp
 $Comp
-L power:GND #PWR?
+L power:GND #PWR0106
 U 1 1 6048CE5C
 P 3800 5400
-F 0 "#PWR?" H 3800 5150 50  0001 C CNN
+F 0 "#PWR0106" H 3800 5150 50  0001 C CNN
 F 1 "GND" H 3805 5227 50  0000 C CNN
 F 2 "" H 3800 5400 50  0001 C CNN

Commit message: reset button + per key leds
Parts:
- removed J1, J2: Conn_01x12, Connector_PinHeader_2.54mm:PinHeader_1x12_P2.54mm_Vertical, symbol Connector_Generic:Conn_01x12
- added D12, D13, D14, D15, D16, D17, D18, D19, D20, D21, D22, D23, D24, D25, D26, D27, D28, D29, D30, D31, D32: SK6812MINI, LED_SMD:LED_SK6812MINI_PLCC4_3.5x3.5mm_P1.75mm, symbol LED:SK6812MINI
- added SW22: SW_Push, Keebio-Parts:SW_Tactile_SPST_Angled_MJTP1117, symbol Switch:SW_Push
- added U1: Elite-C, Keebio-Parts:Elite-C-castellated-24pin-holes, symbol keebio:Elite-C
Connections:
- net labels added: LED
- wire segments 80 -> 181
Other:
- moved on the sheet: J3
